Commit message: added gazebo launch

File: src/tetra_description/urdf/simple_dexter_driveTrain.xacro (robot description, xacro)
@@ -1,8 +1,8 @@
 <?xml version="1.0" ?>
-<robot name="tetra" xmlns:xacro="http://www.ros.org/wiki/xacro">
-<xacro:include filename="$(find tetra_description)/urdf/materials.xacro" />
-<xacro:include filename="$(find tetra_description)/urdf/simple_dexter_driveTrain.trans" />
-<xacro:include filename="$(find tetra_description)/urdf/simple_dexter_driveTrain.gazebo" />
-<link name="world">
+<robot name="tetra_description" xmlns:xacro="http://www.ros.org/wiki/xacro">
+<xacro:include filename="materials.xacro" />
+<xacro:include filename="simple_dexter_driveTrain.trans"/>
+<xacro:include filename="simple_dexter_driveTrain.gazebo"/>
+<link name="dummy">
    </link>
 <link name="base_link">
@@ -15,5 +15,5 @@
     <origin xyz="0 0 0" rpy="0 0 0"/>
     <geometry>
-      <mesh filename="package://tetra_description/meshes/base_link.stl" scale="0.5 0.5 0.5"/>
+      <mesh filename="package://tetra_description/meshes/base_link.stl" scale="0.0254 0.0254 0.0254"/>
     </geometry>
     <material name="silver"/>
@@ -22,5 +22,5 @@
     <origin xyz="0 0 0" rpy="0 0 0"/>
     <geometry>
-      <mesh filename="package://tetra_description/meshes/base_link.stl" scale="0.5 0.5 0.5"/>
+      <mesh filename="package://tetra_description/meshes/base_link.stl" scale="0.0254 0.0254 0.0254"/>
     </geometry>
   </collision>
@@ -35,5 +35,5 @@
     <origin xyz="-0.153738 -0.239644 -0.303299" rpy="0 0 0"/>
     <geometry>
-      <mesh filename="package://tetra_description/meshes/drive_housing_v2_1.stl" scale="0.5 0.5 0.5"/>
+      <mesh filename="package://tetra_description/meshes/drive_housing_v2_1.stl" scale="0.0254 0.0254 0.0254"/>
     </geometry>
     <material name="silver"/>
@@ -42,5 +42,5 @@
     <origin xyz="-0.153738 -0.239644 -0.303299" rpy="0 0 0"/>
     <geometry>
-      <mesh filename="package://tetra_description/meshes/drive_housing_v2_1.stl" scale="0.5 0.5 0.5"/>
+      <mesh filename="package://tetra_description/meshes/drive_housing_v2_1.stl" scale="0.0254 0.0254 0.0254"/>
     </geometry>
   </collision>
@@ -55,5 +55,5 @@
     <origin xyz="0.074862 -0.239644 -0.303299" rpy="0 0 0"/>
     <geometry>
-      <mesh filename="package://tetra_description/meshes/drive_housing_v2__1__1.stl" scale="0.5 0.5 0.5"/>
+      <mesh filename="package://tetra_description/meshes/drive_housing_v2__1__1.stl" scale="0.0254 0.0254 0.0254"/>
     </geometry>
     <material name="silver"/>
@@ -62,5 +62,5 @@
     <origin xyz="0.074862 -0.239644 -0.303299" rpy="0 0 0"/>
     <geometry>
-      <mesh filename="package://tetra_description/meshes/drive_housing_v2__1__1.stl" scale="0.5 0.5 0.5"/>
+      <mesh filename="package://tetra_description/meshes/drive_housing_v2__1__1.stl" scale="0.0254 0.0254 0.0254"/>
     </geometry>
   </collision>
@@ -75,5 +75,5 @@
     <origin xyz="0.239962 -0.493644 -0.175385" rpy="0 0 0"/>
     <geometry>
-      <mesh filename="package://tetra_description/meshes/backFlipper_v2__2__1.stl" scale="0.5 0.5 0.5"/>
+      <mesh filename="package://tetra_description/meshes/backFlipper_v2__2__1.stl" scale="0.0254 0.0254 0.0254"/>
     </geometry>
     <material name="silver"/>
@@ -82,5 +82,5 @@
     <origin xyz="0.239962 -0.493644 -0.175385" rpy="0 0 0"/>
     <geometry>
-      <mesh filename="package://tetra_description/meshes/backFlipper_v2__2__1.stl" scale="0.5 0.5 0.5"/>
+      <mesh filename="package://tetra_description/meshes/backFlipper_v2__2__1.stl" scale="0.0254 0.0254 0.0254"/>
     </geometry>
   </collision>
@@ -95,5 +95,5 @@
     <origin xyz="-0.318838 -0.493644 -0.175385" rpy="0 0 0"/>
     <geometry>
-      <mesh filename="package://tetra_description/meshes/backFlipper_v2__3__1.stl" scale="0.5 0.5 0.5"/>
+      <mesh filename="package://tetra_description/meshes/backFlipper_v2__3__1.stl" scale="0.0254 0.0254 0.0254"/>
     </geometry>
     <material name="silver"/>
@@ -102,5 +102,5 @@
     <origin xyz="-0.318838 -0.493644 -0.175385" rpy="0 0 0"/>
     <geometry>
-      <mesh filename="package://tetra_description/meshes/backFlipper_v2__3__1.stl" scale="0.5 0.5 0.5"/>
+      <mesh filename="package://tetra_description/meshes/backFlipper_v2__3__1.stl" scale="0.0254 0.0254 0.0254"/>
     </geometry>
   </collision>
@@ -115,5 +115,5 @@
     <origin xyz="-0.039438 -0.239644 -0.303299" rpy="0 0 0"/>
     <geometry>
-      <mesh filename="package://tetra_description/meshes/ebox_v1_1.stl" scale="0.5 0.5 0.5"/>
+      <mesh filename="package://tetra_description/meshes/ebox_v1_1.stl" scale="0.0254 0.0254 0.0254"/>
     </geometry>
     <material name="silver"/>
@@ -122,5 +122,5 @@
     <origin xyz="-0.039438 -0.239644 -0.303299" rpy="0 0 0"/>
     <geometry>
-      <mesh filename="package://tetra_description/meshes/ebox_v1_1.stl" scale="0.5 0.5 0.5"/>
+      <mesh filename="package://tetra_description/meshes/ebox_v1_1.stl" scale="0.0254 0.0254 0.0254"/>
     </geometry>
   </collision>
@@ -135,5 +135,5 @@
     <origin xyz="-0.279082 -0.279082 -0.0" rpy="0 0 0"/>
     <geometry>
-      <mesh filename="package://tetra_description/meshes/ARMFINAL_basePlatform_v1_1.stl" scale="0.5 0.5 0.5"/>
+      <mesh filename="package://tetra_description/meshes/ARMFINAL_basePlatform_v1_1.stl" scale="0.0254 0.0254 0.0254"/>
     </geometry>
     <material name="silver"/>
@@ -142,5 +142,5 @@
     <origin xyz="-0.279082 -0.279082 -0.0" rpy="0 0 0"/>
     <geometry>
-      <mesh filename="package://tetra_description/meshes/ARMFINAL_basePlatform_v1_1.stl" scale="0.5 0.5 0.5"/>
+      <mesh filename="package://tetra_description/meshes/ARMFINAL_basePlatform_v1_1.stl" scale="0.0254 0.0254 0.0254"/>
     </geometry>
   </collision>
@@ -155,5 +155,5 @@
     <origin xyz="-0.079182 0.103122 -0.594262" rpy="0 0 0"/>
     <geometry>
-      <mesh filename="package://tetra_description/meshes/ARMFINAL_1401-0043-0032_assembly_v1_1.stl" scale="0.5 0.5 0.5"/>
+      <mesh filename="package://tetra_description/meshes/ARMFINAL_1401-0043-0032_assembly_v1_1.stl" scale="0.0254 0.0254 0.0254"/>
     </geometry>
     <material name="silver"/>
@@ -162,5 +162,5 @@
     <origin xyz="-0.079182 0.103122 -0.594262" rpy="0 0 0"/>
     <geometry>
-      <mesh filename="package://tetra_description/meshes/ARMFINAL_1401-0043-0032_assembly_v1_1.stl" scale="0.5 0.5 0.5"/>
+      <mesh filename="package://tetra_description/meshes/ARMFINAL_1401-0043-0032_assembly_v1_1.stl" scale="0.0254 0.0254 0.0254"/>
     </geometry>
   </collision>
@@ -175,5 +175,5 @@
     <origin xyz="-0.318838 0.014356 -0.175385" rpy="0 0 0"/>
     <geometry>
-      <mesh filename="package://tetra_description/meshes/backFlipper_v2__1__1.stl" scale="0.5 0.5 0.5"/>
+      <mesh filename="package://tetra_description/meshes/backFlipper_v2__1__1.stl" scale="0.0254 0.0254 0.0254"/>
     </geometry>
     <material name="silver"/>
@@ -182,5 +182,5 @@
     <origin xyz="-0.318838 0.014356 -0.175385" rpy="0 0 0"/>
     <geometry>
-      <mesh filename="package://tetra_description/meshes/backFlipper_v2__1__1.stl" scale="0.5 0.5 0.5"/>
+      <mesh filename="package://tetra_description/meshes/backFlipper_v2__1__1.stl" scale="0.0254 0.0254 0.0254"/>
     </geometry>
   </collision>
@@ -195,5 +195,5 @@
     <origin xyz="0.239962 0.014356 -0.175385" rpy="0 0 0"/>
     <geometry>
-      <mesh filename="package://tetra_description/meshes/backFlipper_v2_1.stl" scale="0.5 0.5 0.5"/>
+      <mesh filename="package://tetra_description/meshes/backFlipper_v2_1.stl" scale="0.0254 0.0254 0.0254"/>
     </geometry>
     <material name="silver"/>
@@ -202,5 +202,5 @@
     <origin xyz="0.239962 0.014356 -0.175385" rpy="0 0 0"/>
     <geometry>
-      <mesh filename="package://tetra_description/meshes/backFlipper_v2_1.stl" scale="0.5 0.5 0.5"/>
+      <mesh filename="package://tetra_description/meshes/backFlipper_v2_1.stl" scale="0.0254 0.0254 0.0254"/>
     </geometry>
   </collision>
@@ -215,5 +215,5 @@
     <origin xyz="-0.290898 0.014356 -0.175385" rpy="0 0 0"/>
     <geometry>
-      <mesh filename="package://tetra_description/meshes/sprocket_v1__2__1.stl" scale="0.5 0.5 0.5"/>
+      <mesh filename="package://tetra_description/meshes/sprocket_v1__2__1.stl" scale="0.0254 0.0254 0.0254"/>
     </geometry>
     <material name="silver"/>
@@ -222,5 +222,5 @@
     <origin xyz="-0.290898 0.014356 -0.175385" rpy="0 0 0"/>
     <geometry>
-      <mesh filename="package://tetra_description/meshes/sprocket_v1__2__1.stl" scale="0.5 0.5 0.5"/>
+      <mesh filename="package://tetra_description/meshes/sprocket_v1__2__1.stl" scale="0.0254 0.0254 0.0254"/>
     </geometry>
   </collision>
@@ -235,5 +235,5 @@
     <origin xyz="-0.290898 -0.493644 -0.175385" rpy="0 0 0"/>
     <geometry>
-      <mesh filename="package://tetra_description/meshes/sprocket_v1__1__1.stl" scale="0.5 0.5 0.5"/>
+      <mesh filename="package://tetra_description/meshes/sprocket_v1__1__1.stl" scale="0.0254 0.0254 0.0254"/>
     </geometry>
     <material name="silver"/>
@@ -242,5 +242,5 @@
     <origin xyz="-0.290898 -0.493644 -0.175385" rpy="0 0 0"/>
     <geometry>
-      <mesh filename="package://tetra_description/meshes/sprocket_v1__1__1.stl" scale="0.5 0.5 0.5"/>
+      <mesh filename="package://tetra_description/meshes/sprocket_v1__1__1.stl" scale="0.0254 0.0254 0.0254"/>
     </geometry>
   </collision>
@@ -255,5 +255,5 @@
     <origin xyz="0.212022 -0.493644 -0.175385" rpy="0 0 0"/>
     <geometry>
-      <mesh filename="package://tetra_description/meshes/sprocket_v1_1.stl" scale="0.5 0.5 0.5"/>
+      <mesh filename="package://tetra_description/meshes/sprocket_v1_1.stl" scale="0.0254 0.0254 0.0254"/>
     </geometry>
     <material name="silver"/>
@@ -262,5 +262,5 @@
     <origin xyz="0.212022 -0.493644 -0.175385" rpy="0 0 0"/>
     <geometry>
-      <mesh filename="package://tetra_description/meshes/sprocket_v1_1.stl" scale="0.5 0.5 0.5"/>
+      <mesh filename="package://tetra_description/meshes/sprocket_v1_1.stl" scale="0.0254 0.0254 0.0254"/>
     </geometry>
   </collision>
@@ -275,5 +275,5 @@
     <origin xyz="0.212022 0.014356 -0.175385" rpy="0 0 0"/>
     <geometry>
-      <mesh filename="package://tetra_description/meshes/sprocket_v1__3__1.stl" scale="0.5 0.5 0.5"/>
+      <mesh filename="package://tetra_description/meshes/sprocket_v1__3__1.stl" scale="0.0254 0.0254 0.0254"/>
     </geometry>
     <material name="silver"/>
@@ -282,5 +282,5 @@
     <origin xyz="0.212022 0.014356 -0.175385" rpy="0 0 0"/>
     <geometry>
-      <mesh filename="package://tetra_description/meshes/sprocket_v1__3__1.stl" scale="0.5 0.5 0.5"/>
+      <mesh filename="package://tetra_description/meshes/sprocket_v1__3__1.stl" scale="0.0254 0.0254 0.0254"/>
     </geometry>
   </collision>
@@ -295,5 +295,5 @@
     <origin xyz="0.000818 -0.031548 -0.543579" rpy="0 0 0"/>
     <geometry>
-      <mesh filename="package://tetra_description/meshes/ARMFINAL_1516-4008-0800_v1_1.stl" scale="0.5 0.5 0.5"/>
+      <mesh filename="package://tetra_description/meshes/ARMFINAL_1516-4008-0800_v1_1.stl" scale="0.0254 0.0254 0.0254"/>
     </geometry>
     <material name="silver"/>
@@ -302,5 +302,5 @@
     <origin xyz="0.000818 -0.031548 -0.543579" rpy="0 0 0"/>
     <geometry>
-      <mesh filename="package://tetra_description/meshes/ARMFINAL_1516-4008-0800_v1_1.stl" scale="0.5 0.5 0.5"/>
+      <mesh filename="package://tetra_description/meshes/ARMFINAL_1516-4008-0800_v1_1.stl" scale="0.0254 0.0254 0.0254"/>
     </geometry>
   </collision>
@@ -315,5 +315,5 @@
     <origin xyz="-0.079182 -0.031548 -0.543579" rpy="0 0 0"/>
     <geometry>
-      <mesh filename="package://tetra_description/meshes/ARMFINAL_LowerArmPlate_v1_1.stl" scale="0.5 0.5 0.5"/>
+      <mesh filename="package://tetra_description/meshes/ARMFINAL_LowerArmPlate_v1_1.stl" scale="0.0254 0.0254 0.0254"/>
     </geometry>
     <material name="silver"/>
@@ -322,5 +322,5 @@
     <origin xyz="-0.079182 -0.031548 -0.543579" rpy="0 0 0"/>
     <geometry>
-      <mesh filename="package://tetra_description/meshes/ARMFINAL_LowerArmPlate_v1_1.stl" scale="0.5 0.5 0.5"/>
+      <mesh filename="package://tetra_description/meshes/ARMFINAL_LowerArmPlate_v1_1.stl" scale="0.0254 0.0254 0.0254"/>
     </geometry>
   </collision>
@@ -335,5 +335,5 @@
     <origin xyz="-0.021726 0.120253 -0.868651" rpy="0 0 0"/>
     <geometry>
-      <mesh filename="package://tetra_description/meshes/ARMFINAL_LowerArmPlate_v1__1__1.stl" scale="0.5 0.5 0.5"/>
+      <mesh filename="package://tetra_description/meshes/ARMFINAL_LowerArmPlate_v1__1__1.stl" scale="0.0254 0.0254 0.0254"/>
     </geometry>
     <material name="silver"/>
@@ -342,5 +342,5 @@
     <origin xyz="-0.021726 0.120253 -0.868651" rpy="0 0 0"/>
     <geometry>
-      <mesh filename="package://tetra_description/meshes/ARMFINAL_LowerArmPlate_v1__1__1.stl" scale="0.5 0.5 0.5"/>
+      <mesh filename="package://tetra_description/meshes/ARMFINAL_LowerArmPlate_v1__1__1.stl" scale="0.0254 0.0254 0.0254"/>
     </geometry>
   </collision>
@@ -355,5 +355,5 @@
     <origin xyz="-0.090238 -0.290444 -0.379499" rpy="0 0 0"/>
     <geometry>
-      <mesh filename="package://tetra_description/meshes/ARMFINAL_baseOuter_v1_1.stl" scale="0.5 0.5 0.5"/>
+      <mesh filename="package://tetra_description/meshes/ARMFINAL_baseOuter_v1_1.stl" scale="0.0254 0.0254 0.0254"/>
     </geometry>
     <material name="silver"/>
@@ -362,5 +362,5 @@
     <origin xyz="-0.090238 -0.290444 -0.379499" rpy="0 0 0"/>
     <geometry>
-      <mesh filename="package://tetra_description/meshes/ARMFINAL_baseOuter_v1_1.stl" scale="0.5 0.5 0.5"/>
+      <mesh filename="package://tetra_description/meshes/ARMFINAL_baseOuter_v1_1.stl" scale="0.0254 0.0254 0.0254"/>
     </geometry>
   </collision>
@@ -375,5 +375,5 @@
     <origin xyz="0.017712 -0.277744 -0.481099" rpy="0 0 0"/>
     <geometry>
-      <mesh filename="package://tetra_description/meshes/ARMFINAL_baseAxle_v1_1.stl" scale="0.5 0.5 0.5"/>
+      <mesh filename="package://tetra_description/meshes/ARMFINAL_baseAxle_v1_1.stl" scale="0.0254 0.0254 0.0254"/>
     </geometry>
     <material name="silver"/>
@@ -382,5 +382,5 @@
     <origin xyz="0.017712 -0.277744 -0.481099" rpy="0 0 0"/>
     <geometry>
-      <mesh filename="package://tetra_description/meshes/ARMFINAL_baseAxle_v1_1.stl" scale="0.5 0.5 0.5"/>
+      <mesh filename="package://tetra_description/meshes/ARMFINAL_baseAxle_v1_1.stl" scale="0.0254 0.0254 0.0254"/>
     </geometry>
   </collision>
@@ -395,5 +395,5 @@
     <origin xyz="0.000818 0.110994 -0.563246" rpy="0 0 0"/>
     <geometry>
-      <mesh filename="package://tetra_description/meshes/ARMFINAL_1401-0043-0032_assembly_v1__1__1.stl" scale="0.5 0.5 0.5"/>
+      <mesh filename="package://tetra_description/meshes/ARMFINAL_1401-0043-0032_assembly_v1__1__1.stl" scale="0.0254 0.0254 0.0254"/>
     </geometry>
     <material name="silver"/>
@@ -402,5 +402,5 @@
     <origin xyz="0.000818 0.110994 -0.563246" rpy="0 0 0"/>
     <geometry>
-      <mesh filename="package://tetra_description/meshes/ARMFINAL_1401-0043-0032_assembly_v1__1__1.stl" scale="0.5 0.5 0.5"/>
+      <mesh filename="package://tetra_description/meshes/ARMFINAL_1401-0043-0032_assembly_v1__1__1.stl" scale="0.0254 0.0254 0.0254"/>
     </geometry>
   </collision>
@@ -415,5 +415,5 @@
     <origin xyz="0.000693 0.091549 -0.574818" rpy="0 0 0"/>
     <geometry>
-      <mesh filename="package://tetra_description/meshes/ARMFINAL_upperArmHinge_v1_1.stl" scale="0.5 0.5 0.5"/>
+      <mesh filename="package://tetra_description/meshes/ARMFINAL_upperArmHinge_v1_1.stl" scale="0.0254 0.0254 0.0254"/>
     </geometry>
     <material name="silver"/>
@@ -422,5 +422,5 @@
     <origin xyz="0.000693 0.091549 -0.574818" rpy="0 0 0"/>
     <geometry>
-      <mesh filename="package://tetra_description/meshes/ARMFINAL_upperArmHinge_v1_1.stl" scale="0.5 0.5 0.5"/>
+      <mesh filename="package://tetra_description/meshes/ARMFINAL_upperArmHinge_v1_1.stl" scale="0.0254 0.0254 0.0254"/>
     </geometry>
   </collision>
@@ -435,5 +435,5 @@
     <origin xyz="0.011362 -0.290444 -0.379499" rpy="0 0 0"/>
     <geometry>
-      <mesh filename="package://tetra_description/meshes/ARMFINAL_baseOuter1_v1_1.stl" scale="0.5 0.5 0.5"/>
+      <mesh filename="package://tetra_description/meshes/ARMFINAL_baseOuter1_v1_1.stl" scale="0.0254 0.0254 0.0254"/>
     </geometry>
     <material name="silver"/>
@@ -442,12 +442,12 @@
     <origin xyz="0.011362 -0.290444 -0.379499" rpy="0 0 0"/>
     <geometry>
-      <mesh filename="package://tetra_description/meshes/ARMFINAL_baseOuter1_v1_1.stl" scale="0.5 0.5 0.5"/>
-    </geometry>
-  </collision>
-</link>
-  <joint name="dummy_joint" type="fixed">
-     <parent link="world"/>
-     <child link="base_link"/>
-   </joint>
+      <mesh filename="package://tetra_description/meshes/ARMFINAL_baseOuter1_v1_1.stl" scale="0.0254 0.0254 0.0254"/>
+    </geometry>
+  </collision>
+</link>
+<joint name="dummy_joint" type="fixed">
+  <parent link="dummy"/>
+  <child link="base_link"/>
+</joint>
 <joint name="Rigid 1" type="fixed">
   <origin xyz="0.153738 0.239644 0.303299" rpy="0 0 0"/>
@@ -460,10 +460,9 @@
   <child link="drive_housing_v2__1__1"/>
 </joint>
-<joint name="Revolute 6" type="revolute">
+<joint name="Revolute 6" type="continuous">
   <origin xyz="-0.1651 0.254 -0.127914" rpy="0 0 0"/>
   <parent link="drive_housing_v2__1__1"/>
   <child link="backFlipper_v2__2__1"/>
-  <axis xyz="-0.1651 0 -0.127914"/>
-  <limit effort="1000.0" lower="0.0" upper="0.548" velocity="0.5"/>
+  <axis xyz="1.0 0.0 0.0"/>
 </joint>
 <joint name="Revolute 7" type="continuous">
@@ -492,5 +491,5 @@
   <parent link="drive_housing_v2_1"/>
   <child link="backFlipper_v2__1__1"/>
-  <axis xyz="1.0 0.0 0.0"/>
+  <axis xyz="1.0 -0.0 0.0"/>
 </joint>
 <joint name="Revolute 38" type="continuous">

File: src/tetra_description/urdf/test.urdf (robot description, URDF)
Before this commit: robot tetra, 2 links, 1 joints
Links:
- removed link world
- added link right_leg; visual box size=0.6 0.1 0.2
- link base_link: mass 63.29011858080009 -> None; geometry visual cylinder length=0.6 radius=0.2
Joints:
- removed joint dummy_joint
- added joint base_to_right_leg: type fixed, parent base_link, child right_leg
