Commit message: updated urdf and made gazebo launch file

File: install/test_bot/share/test_bot/description/lidar.xacro (robot description, xacro)
@@ -1,8 +1,8 @@
 <?xml version="1.0"?>
-<robot xmlns:xacro="http://www.ros.org/wiki/xacro"  name="robot">
-    <joint name = "laser_joint" type = "continous">
+<robot xmlns:xacro="http://www.ros.org/wiki/xacro">
+    <joint name = "laser_joint" type = "fixed">
         <parent link = "chassis"/>
         <child link = "laser_frame"/>
-        <origin xyz= "0.1 0 0.14" rpy "0 0 0"/> <!-- check this since the lidar spins-->
+        <origin xyz= "0.3 0 0.14" rpy="0 0 0"/> <!-- check this since the lidar spins-->
     </joint>
     <link name = "laser_frame">

File: install/test_bot/share/test_bot/description/robot_core.xacro (robot description, xacro)
@@ -88,5 +88,4 @@
     </link>
     <!-- CASTER WHEEL LINK -->
-<!--
     <joint name="caster_wheel_joint" type="fixed">
         <parent link="chassis"/>
@@ -110,4 +109,3 @@
         </xacro:inertial_sphere>
     </link>
-     -->
 </robot>

File: test_bot/description/robot_core.xacro (robot description, xacro)
@@ -41,15 +41,18 @@
         </xacro:inertial_box>
     </link>
+    <gazebo>
+        <material>Gazebo/White</material>
+    </gazebo>
     <!-- LEFT WHEEL LINK -->
-    <joint name="left_wheel_joint" type="continuous">
+    <joint name="front_left_wheel_joint" type="continuous">
         <parent link="base_link"/>
-        <child link="left_wheel"/>
-        <origin xyz="0 0.39 0" rpy="-${pi/2} 0 0" />
+        <child link="front_left_wheel"/>
+        <origin xyz="0.25 0.35 0" rpy="-${pi/2} 0 0" />
         <axis xyz="0 0 1"/>
     </joint>
-    <link name="left_wheel">
+    <link name="front_left_wheel">
         <visual>
             <geometry>
-                <cylinder radius="0.15" length="0.18"/>
+                <cylinder radius="0.1" length="0.1"/>
             </geometry>
             <material name="blue"/>
@@ -57,22 +60,27 @@
         <collision>
             <geometry>
-                <cylinder radius="0.15" length="0.18"/>
+                <cylinder radius="0.1" length="0.1"/>
             </geometry>
         </collision>
-        <xacro:inertial_cylinder mass="0.1" length="0.18" radius="0.15">
+        <xacro:inertial_cylinder mass="0.1" length="0.1" radius="0.1">
             <origin xyz="0 0 0" rpy="0 0 0"/>
         </xacro:inertial_cylinder>
     </link>
+     <gazebo>
+        <material>Gazebo/Blue</material>
+        <mu1 value="0.0001"/>
+        <mu2 value="0.0001"/>
+    </gazebo>
     <!-- RIGHT WHEEL LINK -->
-    <joint name="right_wheel_joint" type="continuous">
+    <joint name="front_right_wheel_joint" type="continuous">
         <parent link="base_link"/>
-        <child link="right_wheel"/>
-        <origin xyz="0 -0.39 0" rpy="${pi/2} 0 0" />
+        <child link="front_right_wheel"/>
+        <origin xyz="0.25 -0.35 0" rpy="${pi/2} 0 0" />
         <axis xyz="0 0 -1"/>
     </joint>
-    <link name="right_wheel">
+    <link name="front_right_wheel">
         <visual>
             <geometry>
-                <cylinder radius="0.15" length="0.18"/>
+                <cylinder radius="0.1" length="0.1"/>
             </geometry>
             <material name="blue"/>
@@ -80,17 +88,72 @@
         <collision>
             <geometry>
-                <cylinder radius="0.15" length="0.18"/>
+                <cylinder radius="0.1" length="0.1"/>
             </geometry>
         </collision>
-        <xacro:inertial_cylinder mass="0.1" length="0.18" radius="0.15">
+        <xacro:inertial_cylinder mass="0.1" length="0.1" radius="0.1">
             <origin xyz="0 0 0" rpy="0 0 0"/>
         </xacro:inertial_cylinder>
     </link>
+     <gazebo>
+        <material>Gazebo/Blue</material>
+        <mu1 value="0.0001"/>
+        <mu2 value="0.0001"/>
+    </gazebo>
+    <joint name="back_left_wheel_joint" type="continuous">
+        <parent link="base_link"/>
+        <child link="back_left_wheel"/>
+        <origin xyz="-0.25 0.35 0" rpy="-${pi/2} 0 0" />
+        <axis xyz="0 0 1"/>
+    </joint>
+    <link name="back_left_wheel">
+        <visual>
+            <geometry>
+                <cylinder radius="0.1" length="0.1"/>
+            </geometry>
+            <material name="blue"/>
+        </visual>
+        <collision>
+            <geometry>
+                <cylinder radius="0.1" length="0.1"/>
+            </geometry>
+        </collision>
+        <xacro:inertial_cylinder mass="0.1" length="0.1" radius="0.1">
+            <origin xyz="0 0 0" rpy="0 0 0"/>
+        </xacro:inertial_cylinder>
+    </link>
+    <gazebo>
+        <material>Gazebo/Blue</material>
+    </gazebo>
+    <!-- RIGHT WHEEL LINK -->
+    <joint name="back_right_wheel_joint" type="continuous">
+        <parent link="base_link"/>
+        <child link="back_right_wheel"/>
+        <origin xyz="-0.25 -0.35 0" rpy="${pi/2} 0 0" />
+        <axis xyz="0 0 -1"/>
+    </joint>
+    <link name="back_right_wheel">
+        <visual>
+            <geometry>
+                <cylinder radius="0.1" length="0.1"/>
+            </geometry>
+            <material name="blue"/>
+        </visual>
+        <collision>
+            <geometry>
+                <cylinder radius="0.1" length="0.1"/>
+            </geometry>
+        </collision>
+        <xacro:inertial_cylinder mass="0.1" length="0.1" radius="0.1">
+            <origin xyz="0 0 0" rpy="0 0 0"/>
+        </xacro:inertial_cylinder>
+    </link>
+    <gazebo>
+        <material>Gazebo/Blue</material>
+    </gazebo>
     <!-- CASTER WHEEL LINK -->
-<!--
-    <joint name="caster_wheel_joint" type="fixed">
+    <!-- <joint name="caster_wheel_joint" type="fixed">
         <parent link="chassis"/>
         <child link="caster_wheel"/>
-        <origin xyz="0.24 0 0"/>
+        <origin xyz="0.48 0 0"/>
     </joint>
     <link name="caster_wheel">
@@ -109,5 +172,4 @@
             <origin xyz="0 0 0" rpy="0 0 0"/>
         </xacro:inertial_sphere>
-    </link>
-     -->
+    </link> -->
 </robot>

File: test_bot/install/test_bot/share/test_bot/description/robot_core.xacro (robot description, xacro)
@@ -42,14 +42,14 @@
     </link>
     <!-- LEFT WHEEL LINK -->
-    <joint name="left_wheel_joint" type="continuous">
+    <joint name="front_left_wheel_joint" type="continuous">
         <parent link="base_link"/>
-        <child link="left_wheel"/>
-        <origin xyz="0 0.39 0" rpy="-${pi/2} 0 0" />
+        <child link="front_left_wheel"/>
+        <origin xyz="0.25 0.35 0" rpy="-${pi/2} 0 0" />
         <axis xyz="0 0 1"/>
     </joint>
-    <link name="left_wheel">
+    <link name="front_left_wheel">
         <visual>
             <geometry>
-                <cylinder radius="0.15" length="0.18"/>
+                <cylinder radius="0.1" length="0.1"/>
             </geometry>
             <material name="blue"/>
@@ -57,22 +57,22 @@
         <collision>
             <geometry>
-                <cylinder radius="0.15" length="0.18"/>
+                <cylinder radius="0.1" length="0.1"/>
             </geometry>
         </collision>
-        <xacro:inertial_cylinder mass="0.1" length="0.18" radius="0.15">
+        <xacro:inertial_cylinder mass="0.1" length="0.1" radius="0.1">
             <origin xyz="0 0 0" rpy="0 0 0"/>
         </xacro:inertial_cylinder>
     </link>
     <!-- RIGHT WHEEL LINK -->
-    <joint name="right_wheel_joint" type="continuous">
+    <joint name="front_right_wheel_joint" type="continuous">
         <parent link="base_link"/>
-        <child link="right_wheel"/>
-        <origin xyz="0 -0.39 0" rpy="${pi/2} 0 0" />
+        <child link="front_right_wheel"/>
+        <origin xyz="0.25 -0.35 0" rpy="${pi/2} 0 0" />
         <axis xyz="0 0 -1"/>
     </joint>
-    <link name="right_wheel">
+    <link name="front_right_wheel">
         <visual>
             <geometry>
-                <cylinder radius="0.15" length="0.18"/>
+                <cylinder radius="0.1" length="0.1"/>
             </geometry>
             <material name="blue"/>
@@ -80,17 +80,61 @@
         <collision>
             <geometry>
-                <cylinder radius="0.15" length="0.18"/>
+                <cylinder radius="0.1" length="0.1"/>
             </geometry>
         </collision>
-        <xacro:inertial_cylinder mass="0.1" length="0.18" radius="0.15">
+        <xacro:inertial_cylinder mass="0.1" length="0.1" radius="0.1">
+            <origin xyz="0 0 0" rpy="0 0 0"/>
+        </xacro:inertial_cylinder>
+    </link>
+    <joint name="back_left_wheel_joint" type="continuous">
+        <parent link="base_link"/>
+        <child link="back_left_wheel"/>
+        <origin xyz="-0.25 0.35 0" rpy="-${pi/2} 0 0" />
+        <axis xyz="0 0 1"/>
+    </joint>
+    <link name="back_left_wheel">
+        <visual>
+            <geometry>
+                <cylinder radius="0.1" length="0.1"/>
+            </geometry>
+            <material name="blue"/>
+        </visual>
+        <collision>
+            <geometry>
+                <cylinder radius="0.1" length="0.1"/>
+            </geometry>
+        </collision>
+        <xacro:inertial_cylinder mass="0.1" length="0.1" radius="0.1">
+            <origin xyz="0 0 0" rpy="0 0 0"/>
+        </xacro:inertial_cylinder>
+    </link>
+    <!-- RIGHT WHEEL LINK -->
+    <joint name="back_right_wheel_joint" type="continuous">
+        <parent link="base_link"/>
+        <child link="back_right_wheel"/>
+        <origin xyz="-0.25 -0.35 0" rpy="${pi/2} 0 0" />
+        <axis xyz="0 0 -1"/>
+    </joint>
+    <link name="back_right_wheel">
+        <visual>
+            <geometry>
+                <cylinder radius="0.1" length="0.1"/>
+            </geometry>
+            <material name="blue"/>
+        </visual>
+        <collision>
+            <geometry>
+                <cylinder radius="0.1" length="0.1"/>
+            </geometry>
+        </collision>
+        <xacro:inertial_cylinder mass="0.1" length="0.1" radius="0.1">
             <origin xyz="0 0 0" rpy="0 0 0"/>
         </xacro:inertial_cylinder>
     </link>
     <!-- CASTER WHEEL LINK -->
-<!--
-    <joint name="caster_wheel_joint" type="fixed">
+    <!-- <joint name="caster_wheel_joint" type="fixed">
         <parent link="chassis"/>
         <child link="caster_wheel"/>
-        <origin xyz="0.24 0 0"/>
+        <origin xyz="0.48 0 0"/>
     </joint>
     <link name="caster_wheel">
@@ -109,5 +153,4 @@
             <origin xyz="0 0 0" rpy="0 0 0"/>
         </xacro:inertial_sphere>
-    </link>
-     -->
+    </link> -->
 </robot>
